Commit message: update xacro files

File: custom_sawyer_description/urdf/sawyer.urdf.xacro (robot description, xacro)
@@ -6,10 +6,10 @@
   <xacro:arg name="electric_gripper" default="false"/>
   <!-- Sawyer Base URDF -->
-  <xacro:include filename="$(find sawyer_description)/urdf/sawyer_base.urdf.xacro">
+  <xacro:include filename="$(find custom_sawyer_description)/urdf/sawyer_base.urdf.xacro">
     <xacro:arg name="gazebo" value="${gazebo}"/>
     <xacro:arg name="pedestal" value="${pedestal}"/>
   </xacro:include>
   <xacro:if value="$(arg gazebo)">
-  <xacro:include filename="$(find sawyer_description)/urdf/sawyer_base.gazebo.xacro">
+  <xacro:include filename="$(find custom_sawyer_description)/urdf/sawyer_base.gazebo.xacro">
     <xacro:arg name="static" value="${static}"/>
     <xacro:arg name="pedestal" value="${pedestal}"/>
@@ -18,5 +18,5 @@
   <!-- Electric Gripper End Effector -->
   <xacro:if value="$(arg electric_gripper)">
-  <xacro:include filename="$(find sawyer_description)/urdf/sawyer_electric_gripper.urdf.xacro">
+  <xacro:include filename="$(find custom_sawyer_description)/urdf/sawyer_electric_gripper.urdf.xacro">
     <xacro:arg name="gazebo" value="${gazebo}"/>
   </xacro:include>

File: custom_sawyer_description/urdf/sawyer_base.urdf.xacro (robot description, xacro)
@@ -42,5 +42,5 @@
       <origin rpy="1.57079632679 0 -1.57079632679" xyz="0.26 0.345 -0.91488"/>
       <geometry>
-        <mesh filename="package://sawyer_description/meshes/sawyer_pv/pedestal.DAE"/>
+        <mesh filename="package://custom_sawyer_description/meshes/sawyer_pv/pedestal.DAE"/>
       </geometry>
       <material name="darkgray"/>
@@ -109,5 +109,5 @@
       <origin rpy="0 0 0" xyz="0 0 0"/>
       <geometry>
-        <mesh filename="package://sawyer_description/meshes/sawyer_pv/base.DAE"/>
+        <mesh filename="package://custom_sawyer_description/meshes/sawyer_pv/base.DAE"/>
       </geometry>
       <material name="sawyer_red"/>
@@ -129,5 +129,5 @@
       <origin rpy="0 0 0" xyz="0 0 0"/>
       <geometry>
-        <mesh filename="package://sawyer_description/meshes/sawyer_mp3/l0.DAE"/>
+        <mesh filename="package://custom_sawyer_description/meshes/sawyer_mp3/l0.DAE"/>
       </geometry>
       <material name="sawyer_red"/>
@@ -159,5 +159,5 @@
       <origin rpy="0 0 0" xyz="0 0 0"/>
       <geometry>
-        <mesh filename="package://sawyer_description/meshes/sawyer_pv/head.DAE"/>
+        <mesh filename="package://custom_sawyer_description/meshes/sawyer_pv/head.DAE"/>
       </geometry>
       <material name="sawyer_red"/>
@@ -204,5 +204,5 @@
       <origin rpy="0 0 0" xyz="0 0 0"/>
       <geometry>
-        <mesh filename="package://sawyer_description/meshes/sawyer_mp3/l1.DAE"/>
+        <mesh filename="package://custom_sawyer_description/meshes/sawyer_mp3/l1.DAE"/>
       </geometry>
       <material name="sawyer_red"/>
@@ -234,5 +234,5 @@
       <origin rpy="0 0 0" xyz="0 0 0"/>
       <geometry>
-        <mesh filename="package://sawyer_description/meshes/sawyer_pv/l2.DAE"/>
+        <mesh filename="package://custom_sawyer_description/meshes/sawyer_pv/l2.DAE"/>
       </geometry>
       <material name="sawyer_red"/>
@@ -264,5 +264,5 @@
       <origin rpy="0 0 0" xyz="0 0 0"/>
       <geometry>
-        <mesh filename="package://sawyer_description/meshes/sawyer_pv/l3.DAE"/>
+        <mesh filename="package://custom_sawyer_description/meshes/sawyer_pv/l3.DAE"/>
       </geometry>
       <material name="sawyer_red"/>
@@ -294,5 +294,5 @@
       <origin rpy="0 0 0" xyz="0 0 0"/>
       <geometry>
-        <mesh filename="package://sawyer_description/meshes/sawyer_pv/l4.DAE"/>
+        <mesh filename="package://custom_sawyer_description/meshes/sawyer_pv/l4.DAE"/>
       </geometry>
       <material name="sawyer_red"/>
@@ -339,5 +339,5 @@
       <origin rpy="0 0 0" xyz="0 0 0"/>
       <geometry>
-        <mesh filename="package://sawyer_description/meshes/sawyer_pv/l5.DAE"/>
+        <mesh filename="package://custom_sawyer_description/meshes/sawyer_pv/l5.DAE"/>
       </geometry>
       <material name="sawyer_red"/>
@@ -383,5 +383,5 @@
       <origin rpy="0 0 0" xyz="0 0 0"/>
       <geometry>
-        <mesh filename="package://sawyer_description/meshes/sawyer_mp1/l6.DAE"/>
+        <mesh filename="package://custom_sawyer_description/meshes/sawyer_mp1/l6.DAE"/>
       </geometry>
       <material name="sawyer_red"/>

File: custom_sawyer_description/urdf/sawyer_base_fixed.urdf.xacro (robot description, xacro)
@@ -42,5 +42,5 @@
       <origin rpy="1.57079632679 0 -1.57079632679" xyz="0.26 0.345 -0.91488"/>
       <geometry>
-        <mesh filename="package://sawyer_description/meshes/sawyer_pv/pedestal.DAE"/>
+        <mesh filename="package://custom_sawyer_description/meshes/sawyer_pv/pedestal.DAE"/>
       </geometry>
       <material name="darkgray"/>
@@ -109,5 +109,5 @@
       <origin rpy="0 0 0" xyz="0 0 0"/>
       <geometry>
-        <mesh filename="package://sawyer_description/meshes/sawyer_pv/base.DAE"/>
+        <mesh filename="package://custom_sawyer_description/meshes/sawyer_pv/base.DAE"/>
       </geometry>
       <material name="sawyer_red"/>
@@ -129,5 +129,5 @@
       <origin rpy="0 0 0" xyz="0 0 0"/>
       <geometry>
-        <mesh filename="package://sawyer_description/meshes/sawyer_mp3/l0.DAE"/>
+        <mesh filename="package://custom_sawyer_description/meshes/sawyer_mp3/l0.DAE"/>
       </geometry>
       <material name="sawyer_red"/>
@@ -159,5 +159,5 @@
       <origin rpy="0 0 0" xyz="0 0 0"/>
       <geometry>
-        <mesh filename="package://sawyer_description/meshes/sawyer_pv/head.DAE"/>
+        <mesh filename="package://custom_sawyer_description/meshes/sawyer_pv/head.DAE"/>
       </geometry>
       <material name="sawyer_red"/>
@@ -204,5 +204,5 @@
       <origin rpy="0 0 0" xyz="0 0 0"/>
       <geometry>
-        <mesh filename="package://sawyer_description/meshes/sawyer_mp3/l1.DAE"/>
+        <mesh filename="package://custom_sawyer_description/meshes/sawyer_mp3/l1.DAE"/>
       </geometry>
       <material name="sawyer_red"/>
@@ -234,5 +234,5 @@
       <origin rpy="0 0 0" xyz="0 0 0"/>
       <geometry>
-        <mesh filename="package://sawyer_description/meshes/sawyer_pv/l2.DAE"/>
+        <mesh filename="package://custom_sawyer_description/meshes/sawyer_pv/l2.DAE"/>
       </geometry>
       <material name="sawyer_red"/>
@@ -264,5 +264,5 @@
       <origin rpy="0 0 0" xyz="0 0 0"/>
       <geometry>
-        <mesh filename="package://sawyer_description/meshes/sawyer_pv/l3.DAE"/>
+        <mesh filename="package://custom_sawyer_description/meshes/sawyer_pv/l3.DAE"/>
       </geometry>
       <material name="sawyer_red"/>
@@ -294,5 +294,5 @@
       <origin rpy="0 0 0" xyz="0 0 0"/>
       <geometry>
-        <mesh filename="package://sawyer_description/meshes/sawyer_pv/l4.DAE"/>
+        <mesh filename="package://custom_sawyer_description/meshes/sawyer_pv/l4.DAE"/>
       </geometry>
       <material name="sawyer_red"/>
@@ -339,5 +339,5 @@
       <origin rpy="0 0 0" xyz="0 0 0"/>
       <geometry>
-        <mesh filename="package://sawyer_description/meshes/sawyer_pv/l5.DAE"/>
+        <mesh filename="package://custom_sawyer_description/meshes/sawyer_pv/l5.DAE"/>
       </geometry>
       <material name="sawyer_red"/>
@@ -383,5 +383,5 @@
       <origin rpy="0 0 0" xyz="0 0 0"/>
       <geometry>
-        <mesh filename="package://sawyer_description/meshes/sawyer_mp1/l6.DAE"/>
+        <mesh filename="package://custom_sawyer_description/meshes/sawyer_mp1/l6.DAE"/>
       </geometry>
       <material name="sawyer_red"/>

File: custom_sawyer_description/urdf/sawyer_electric_gripper_fixed.urdf.xacro (robot description, xacro)
@@ -8,5 +8,5 @@
     <xacro:property name="gazebo_tag" value="false" scope="local"/>
   </xacro:unless>
-  <xacro:include filename="$(find sawyer_description)/urdf/rethink_electric_gripper_fixed.xacro" />
+  <xacro:include filename="$(find custom_sawyer_description)/urdf/rethink_electric_gripper_fixed.xacro" />
   <xacro:rethink_electric_gripper_fixed side="right"
                                   gazebo="${gazebo_tag}"

File: custom_sawyer_description/urdf/sawyer_fixed.urdf.xacro (robot description, xacro)
@@ -6,10 +6,10 @@
   <xacro:arg name="electric_gripper" default="false"/>
   <!-- Sawyer Base URDF -->
-  <xacro:include filename="$(find sawyer_description)/urdf/sawyer_base_fixed.urdf.xacro">
+  <xacro:include filename="$(find custom_sawyer_description)/urdf/sawyer_base_fixed.urdf.xacro">
     <xacro:arg name="gazebo" value="${gazebo}"/>
     <xacro:arg name="pedestal" value="${pedestal}"/>
   </xacro:include>
   <xacro:if value="$(arg gazebo)">
-  <xacro:include filename="$(find sawyer_description)/urdf/sawyer_base.gazebo.xacro">
+  <xacro:include filename="$(find custom_sawyer_description)/urdf/sawyer_base.gazebo.xacro">
     <xacro:arg name="static" value="${static}"/>
     <xacro:arg name="pedestal" value="${pedestal}"/>
@@ -18,5 +18,5 @@
   <!-- Electric Gripper End Effector -->
   <xacro:if value="$(arg electric_gripper)">
-  <xacro:include filename="$(find sawyer_description)/urdf/sawyer_electric_gripper_fixed.urdf.xacro">
+  <xacro:include filename="$(find custom_sawyer_description)/urdf/sawyer_electric_gripper_fixed.urdf.xacro">
     <xacro:arg name="gazebo" value="${gazebo}"/>
   </xacro:include>
